File: misfits.kicad_sch (KiCad schematic)
At the start: 0 parts

Commit message: Finished schematic
Signed-off-by: Red Lucy <user@domain.tld>
Parts:
- added C1, C10, C12, C13, C14, C15, C16, C17, C18, C2, C3, C8: 1uF, CL10A105KO8NNNC:CAPC1608X90N, symbol CL10A105KO8NNNC:CL10A105KO8NNNC
- added C11, C9: 0.47uF, CL10A475KP8NNNC:CAPC1608X90N, symbol CL10A475KP8NNNC:CL10A475KP8NNNC
- added C4, C6, C7: 0.1uF, CL10B104KA8NNNC:CAPC1608X90N, symbol CL10B104KA8NNNC:CL10B104KA8NNNC
- added C5: 10uF, CL10A106MQ8NNNC:CAPC1608X90N, symbol CL10A106MQ8NNNC:CL10A106MQ8NNNC
- added D1: KT-0603R, KT-0603R:LED_KT-0603R, symbol KT-0603R:KT-0603R
- added D2, D3, D4: B0530W-7-F, B0530W-7-F:SOD3715X145N, symbol B0530W-7-F:B0530W-7-F
- added J1: GT-USB-7010B, GT-USB-7010B:G-SWITCH_GT-USB-7010B, symbol GT-USB-7010B:GT-USB-7010B
- added J2: S2B-PH-K-S_LF__SN_, S2B-PH-K-S_LF__SN_:JST_S2B-PH-K-S_LF__SN_, symbol S2B-PH-K-S_LF__SN_:S2B-PH-K-S_LF__SN_
- added J3: FH34SRJ-24S-0.5SH_50_, FH34SRJ-24S-0.5SH_50_:HRS_FH34SRJ-24S-0.5SH_50_, symbol FH34SRJ-24S-0.5SH_50_:FH34SRJ-24S-0.5SH_50_
- added L1: 47uH 500mA, WE-TPC_4828:WE-TPC_4828, symbol WE-TPC_4828:WE-TPC_4828
- added Q1: 2N7002K-7, 2N7002K-7:SOT91P240X110-3N, symbol 2N7002K-7:2N7002K-7
- added R1, R3, R4: 1k, RC0603JR-071KL:RESC1607X60N, symbol RC0603JR-071KL:RC0603JR-071KL
- added R2: 2k, SMD-RES-2K-1_-1_10W_0603_:R0603, symbol SMD-RES-2K-1_-1_10W_0603_:SMD-RES-2K-1_-1_10W_0603_
- added R5, R7: 1M, RC0603FR-071ML:RESC1607X60N, symbol RC0603FR-071ML:RC0603FR-071ML
- added R6: 200k, RC0603FR-07200KL:RESC1608X60N, symbol RC0603FR-07200KL:RC0603FR-07200KL
- added R8: 2.2k, RC0603JR-072K2L:RESC1608X55N, symbol RC0603JR-072K2L:RC0603JR-072K2L
- added S1: RESET, EVP-AEDB2A:SW_EVP-AEDB2A, symbol EVP-AEDB2A:EVP-AEDB2A
- added S2: BOOT, EVP-AEDB2A:SW_EVP-AEDB2A, symbol EVP-AEDB2A:EVP-AEDB2A
- added U1: ESP32-S3-MINI-1-N8, ESP32-S3-MINI-1-N8:XCVR_ESP32-S3-MINI-1-N8, symbol ESP32-S3-MINI-1-N8:ESP32-S3-MINI-1-N8
- added U2: BQ24040DSQR, BQ24040DSQR:SON40P200X200X80-11N, symbol BQ24040DSQR:BQ24040DSQR
- added U3: TLV75801PDRVR, TLV75801PDRVR:SON65P200X200X80-7N, symbol TLV75801PDRVR:TLV75801PDRVR
- added U4: ESD7104MUTAG, ESD7104MUTAG:IC_ESD7104MUTAG, symbol ESD7104MUTAG:ESD7104MUTAG
Connections:
- new net: C2.1, C3.1, J2.1, R3.1, U2.10 (OUT), U3.4 (EN), U3.6 (IN)
- new net: C12.1, J3.5
- new net: C11.2, D2.A, L1.2, Q1.3
- new net: D1.A, R3.2
- new net: C7.1, S2.2, U1.4 (IO0)
- new net: R5.2, R6.1, U3.2 (FB)
- new net: C6.1, R4.2, S1.2, U1.45 (EN)
- new net: R1.1, U2.2 (ISET)
- new net: R2.1, U2.4 (PRETERM)
- new net: D1.C, U2.8 (~{CHG})
- new net: C13.1, J3.15, J3.16
- new net: C14.1, J3.18
- new net: C15.1, J3.20
- new net: C16.1, J3.22
- new net: C11.1, D3.A, D4.C
- new net 3V3: C4.1, C5.1, C8.1, C9.1, L1.1, R4.1, R5.1, U1.3 (3V3), U3.1 (OUT)
- new net 5V_IN: C1.1, J1.A4_B9 (VBUS_A), J1.B4_A9 (VBUS_B), U2.1 (IN), U4.4 (I/O_4)
- new net BUSY: J3.9, U1.22 (IO18)
- new net CS: J3.12, U1.14 (IO10)
- new net DC: J3.11, U1.13 (IO9)
- new net GDR: J3.2, Q1.1, R7.1
- new net GND: C1.2, C10.2, C12.2, C13.2, C14.2, C15.2, C16.2, C17.2, C18.2, C2.2, C3.2, C4.2, C5.2, C6.2, C7.2, C8.2, C9.2, D3.C, J1.A1_B12 (GND_A), J1.B1_A12 (GND_B), J1.SH1 (SHIELD), J1.SH2 (SHIELD), J1.SH3 (SHIELD), J1.SH4 (SHIELD), J2.2, J3.17, J3.8, J3.S1 (SHIELD), J3.S2 (SHIELD), R1.2, R2.2, R6.2, R7.2, R8.1, S1.1, S1.1_1, S2.1, S2.1_1, U1.1 (GND), U1.2 (GND), U1.42 (GND), U1.43 (GND), U1.46 (GND), U1.47 (GND), U1.48 (GND), U1.49 (GND), U1.50 (GND), U1.51 (GND), U1.52 (GND), U1.53 (GND), U1.54 (GND), U1.55 (GND), U1.56 (GND), U1.57 (GND), U1.58 (GND), U1.59 (GND), U1.60 (GND), U1.61 (GND), U1.61_1 (GND), U1.61_2 (GND), U1.61_3 (GND), U1.61_4 (GND), U1.61_5 (GND), U1.61_6 (GND), U1.61_7 (GND), U1.61_8 (GND), U1.62 (GND), U1.63 (GND), U1.64 (GND), U1.65 (GND), U2.11 (EXP), U2.3 (VSS), U2.7 (ISET2), U3.3 (GND), U4.3 (GND), U4.8 (GND)
- new net PREVGH: C10.1, D2.C, J3.21
- new net PREVGL: C17.1, D4.A, J3.23
- new net RES: J3.10, U1.12 (IO8)
- new net RESE: J3.3, Q1.2, R8.2
- new net SCLK: J3.13, U1.16 (IO12)
- new net SDI: J3.14, U1.15 (IO11)
- new net USB_D_N: J1.A7 (D1-), J1.B7 (D2-), U1.23 (IO19), U4.1 (I/O_1)
- new net USB_D_P: J1.A6 (D1+), J1.B6 (D2+), U1.24 (IO20), U4.2 (I/O_2)
- new net VCOM: C18.1, J3.24
- no-connect marks 0 -> 43
Other:
- note added: "Battery charging"
- note added: "Boot/Reset buttons"
- note added: "ESD protection"
- note added: "USB-C connector (Power-Input and USB-Data)"
- note added: "Voltage regulator (VBUS/BAT_OUT to 3V3)"
- note added: "eInk Panel power delivery"

Commit message: Revision 1 finished
Signed-off-by: Red Lucy <user@domain.tld>
Parts:
- added S3: SETTING1, EVP-AEDB2A:SW_EVP-AEDB2A, symbol EVP-AEDB2A:EVP-AEDB2A
- added S4: SETTING2, EVP-AEDB2A:SW_EVP-AEDB2A, symbol EVP-AEDB2A:EVP-AEDB2A
Connections:
- net at U1.28 (IO33): now also S3.1, S3.1_1
- net at U1.29 (IO34): now also S3.2
- net at U1.31 (IO35): now also S4.1, S4.1_1
- net at U1.32 (IO36): now also S4.2
- no-connect marks 43 -> 39
